File: pcb/mega/stepper_controller_mega.kicad_pcb (KiCad board)
At the start: 2 copper layers, 118.1 x 55.1 mm, 58 parts, among them P1 PWR_JACK_2.5x5.5, P10 HEADER_02X08_SMD, P11 HEADER_02X08_SMD, P2 HEADER_01X03_SMD_RA, P3 HEADER_01X03_SMD_RA, P4 HEADER_01X03_SMD_RA, P5 HEADER_01X03_SMD_RA, P6 HEADER_01X02_SMD_RA, P7 BNC_DOUBLE_RA, P8 HEADER_02X08_SMD, P9 HEADER_02X08_SMD, SW1 SPST_SLIDE_AS, U1 TLE7230R, U2 TLE7230R, U3 TLE7230R, U4 TLE7230R

Commit message: Created stepper_controller_mega.
Parts:
- ARDUINO1: footprint stepper_controller:ARDUINO_MEGA_SHIELD -> stepper_controller_mega:ARDUINO_MEGA_SHIELD
- C1, C2, C3, C4, C5, C6, C7: footprint stepper_controller:SM1210 -> stepper_controller_mega:SM1210
- D1, D10, D11, D12, D13, D14, D15, D16, D17, D18, D19, D2, D20, D21, D22, D23, D24, D25, D26, D27, D28, D29, D3, D30, D31, D32, D33, D4, D5, D6, D7, D8, D9: footprint stepper_controller:LED_555-3XXX -> stepper_controller_mega:LED_555-3XXX
- P1: footprint stepper_controller:DCJACK_2PIN_HIGHCURRENT -> stepper_controller_mega:DCJACK_2PIN_HIGHCURRENT
- P10, P11, P8, P9: footprint stepper_controller:HEADER_02x08_SMD -> stepper_controller_mega:HEADER_02x08_SMD
- P2, P3, P4, P5: footprint stepper_controller:Header_3_Pin_SMD_RA -> stepper_controller_mega:Header_3_Pin_SMD_RA
- P6: footprint stepper_controller:Header_2_Pin_SMD_RA -> stepper_controller_mega:Header_2_Pin_SMD_RA
- P7: footprint stepper_controller:BNC_DOUBLE -> stepper_controller_mega:BNC_DOUBLE
- REG1: footprint stepper_controller:DC_DC_CONV_R78C -> stepper_controller_mega:DC_DC_CONV_R78C
- SW1: footprint stepper_controller:SPST_SLIDE_AS -> stepper_controller_mega:SPST_SLIDE_AS
- U1, U2, U3, U4: footprint stepper_controller:PG-DSO-36 -> stepper_controller_mega:PG-DSO-36
Other:
- board text added: "Janelia Modular Device stepper_controller_mega model_number: 1140 03/2016 ver 1.0"
- board text removed: "Janelia Modular Device stepper_controller model_number: 1140 03/2016 ver 1.0"
