File: pcb/mega/stepper_controller_mega.sch (KiCad schematic (older format))
At the start: 17 parts, among them P1 PWR_JACK_2.5x5.5, P2 HEADER_01X03_SMD_RA, P3 HEADER_01X03_SMD_RA, P4 HEADER_01X03_SMD_RA, P5 HEADER_01X03_SMD_RA, P6 HEADER_01X02_SMD_RA, P7 BNC_DOUBLE_RA, SW1 SPST_SLIDE_AS

Commit message: Created stepper_controller_mega.
Parts:
- ARDUINO1: footprint stepper_controller:ARDUINO_MEGA_SHIELD -> stepper_controller_mega:ARDUINO_MEGA_SHIELD
- C1, C2, C3, R1, R2: footprint stepper_controller:SM1210 -> stepper_controller_mega:SM1210
- D1: footprint stepper_controller:LED_555-3XXX -> stepper_controller_mega:LED_555-3XXX
- IM1: footprint stepper_controller:IM483H_IM805H_PR-22 -> stepper_controller_mega:IM483H_IM805H_PR-22
- P1: footprint stepper_controller:DCJACK_2PIN_HIGHCURRENT -> stepper_controller_mega:DCJACK_2PIN_HIGHCURRENT
- P2, P3, P4, P5: footprint stepper_controller:Header_3_Pin_SMD_RA -> stepper_controller_mega:Header_3_Pin_SMD_RA
- P6: footprint stepper_controller:Header_2_Pin_SMD_RA -> stepper_controller_mega:Header_2_Pin_SMD_RA
- P7: footprint stepper_controller:BNC_DOUBLE -> stepper_controller_mega:BNC_DOUBLE
- REG1: footprint stepper_controller:DC_DC_CONV_R78C -> stepper_controller_mega:DC_DC_CONV_R78C
- SW1: footprint stepper_controller:SPST_SLIDE_AS -> stepper_controller_mega:SPST_SLIDE_AS
Changed lines of the file:
@@
 EESchema Schematic File Version 2
-LIBS:stepper_controller-rescue
+LIBS:stepper_controller_mega-rescue
 LIBS:power
 LIBS:device
@@
 LIBS:contrib
 LIBS:valves
-LIBS:stepper_controller
+LIBS:stepper_controller_mega
 LIBS:components
-LIBS:stepper_controller-cache
+LIBS:stepper_controller_mega-cache
 EELAYER 25 0
 EELAYER END
@@
 encoding utf-8
 Sheet 1 1
-Title "stepper_controller"
+Title "stepper_controller_mega"
 Date ""
 Rev "1.0"
@@
 F 0 "P1" H 1275 7725 50  0000 C CNN
 F 1 "PWR_JACK_2.5x5.5" V 1375 7575 50  0000 C CNN
-F 2 "stepper_controller:DCJACK_2PIN_HIGHCURRENT" H 1175 7625 60  0001 C CNN
+F 2 "stepper_controller_mega:DCJACK_2PIN_HIGHCURRENT" H 1175 7625 60  0001 C CNN
 F 3 "" H 1275 7575 60  0000 C CNN
 F 4 "digikey" H 1375 7825 60  0001 C CNN "Vendor"
@@
 F 0 "D1" H 2200 7675 50  0000 C CNN
 F 1 "LED_24V" H 2200 7475 50  0000 C CNN
-F 2 "stepper_controller:LED_555-3XXX" H 2100 7575 60  0001 C CNN
+F 2 "stepper_controller_mega:LED_555-3XXX" H 2100 7575 60  0001 C CNN
 F 3 "" H 2200 7575 60  0000 C CNN
 F 4 "digikey" H 2300 7775 60  0001 C CNN "Vendor"
@@
 F 0 "C2" H 3125 7600 40  0000 L CNN
 F 1 "10uF" H 3131 7415 40  0000 L CNN
-F 2 "stepper_controller:SM1210" H 3163 7350 30  0001 C CNN
+F 2 "stepper_controller_mega:SM1210" H 3163 7350 30  0001 C CNN
 F 3 "" H 3125 7500 60  0000 C CNN
 F 4 "digikey" H 3225 7700 60  0001 C CNN "Vendor"
@@
 F 0 "C3" H 4425 7600 40  0000 L CNN
 F 1 "10uF" H 4431 7415 40  0000 L CNN
-F 2 "stepper_controller:SM1210" H 4463 7350 30  0001 C CNN
+F 2 "stepper_controller_mega:SM1210" H 4463 7350 30  0001 C CNN
 F 3 "" H 4425 7500 60  0000 C CNN
 F 4 "digikey" H 4525 7700 60  0001 C CNN "Vendor"
@@
 F 0 "REG1" H 3975 6950 60  0000 C CNN
 F 1 "CONV_DC_DC_12V_1A" H 3775 7350 60  0000 C CNN
-F 2 "stepper_controller:DC_DC_CONV_R78C" H 3875 6850 60  0001 C CNN
+F 2 "stepper_controller_mega:DC_DC_CONV_R78C" H 3875 6850 60  0001 C CNN
 F 3 "" H 3775 7250 60  0000 C CNN
 F 4 "digikey" H 3775 7050 60  0001 C CNN "Vendor"
@@
 F 0 "ARDUINO1" H 2550 6100 60  0000 C CNN
 F 1 "ARDUINO_MEGA" H 2500 650 60  0000 C CNN
-F 2 "stepper_controller:ARDUINO_MEGA_SHIELD" H 2450 6000 60  0001 C CNN
+F 2 "stepper_controller_mega:ARDUINO_MEGA_SHIELD" H 2450 6000 60  0001 C CNN
 F 3 "" H 2550 6100 60  0000 C CNN
 F 4 "digikey" H 2650 6200 60  0001 C CNN "Vendor"
@@
 F 0 "P7" H 5750 7675 50  0000 C CNN
 F 1 "BNC_DOUBLE_RA" H 5750 7375 50  0000 C CNN
-F 2 "stepper_controller:BNC_DOUBLE" H 5750 6325 60  0001 C CNN
+F 2 "stepper_controller_mega:BNC_DOUBLE" H 5750 6325 60  0001 C CNN
 F 3 "" H 5750 6325 60  0000 C CNN
 F 4 "digikey" H 5850 7775 60  0001 C CNN "Vendor"
@@
 F 0 "P2" H 650 6400 50  0000 C CNN
 F 1 "HEADER_01X03_SMD_RA" V 750 6600 50  0000 C CNN
-F 2 "stepper_controller:Header_3_Pin_SMD_RA" H 550 6700 60  0001 C CNN
+F 2 "stepper_controller_mega:Header_3_Pin_SMD_RA" H 550 6700 60  0001 C CNN
 F 3 "" H 650 6800 60  0000 C CNN
 F 4 "digikey" H 750 6900 60  0001 C CNN "Vendor"
@@
 F 0 "P3" H 1225 6375 50  0000 C CNN
 F 1 "HEADER_01X03_SMD_RA" V 1325 6575 50  0000 C CNN
-F 2 "stepper_controller:Header_3_Pin_SMD_RA" H 1125 6675 60  0001 C CNN
+F 2 "stepper_controller_mega:Header_3_Pin_SMD_RA" H 1125 6675 60  0001 C CNN
 F 3 "" H 1225 6775 60  0000 C CNN
 F 4 "digikey" H 1325 6875 60  0001 C CNN "Vendor"
@@
 F 0 "P4" H 1800 6375 50  0000 C CNN
 F 1 "HEADER_01X03_SMD_RA" V 1900 6575 50  0000 C CNN
-F 2 "stepper_controller:Header_3_Pin_SMD_RA" H 1700 6675 60  0001 C CNN
+F 2 "stepper_controller_mega:Header_3_Pin_SMD_RA" H 1700 6675 60  0001 C CNN
 F 3 "" H 1800 6775 60  0000 C CNN
 F 4 "digikey" H 1900 6875 60  0001 C CNN "Vendor"
@@
 F 0 "P5" H 2375 6350 50  0000 C CNN
 F 1 "HEADER_01X03_SMD_RA" V 2475 6550 50  0000 C CNN
-F 2 "stepper_controller:Header_3_Pin_SMD_RA" H 2275 6650 60  0001 C CNN
+F 2 "stepper_controller_mega:Header_3_Pin_SMD_RA" H 2275 6650 60  0001 C CNN
 F 3 "" H 2375 6750 60  0000 C CNN
 F 4 "digikey" H 2475 6850 60  0001 C CNN "Vendor"
@@
 F 0 "P6" H 2950 6400 50  0000 C CNN
 F 1 "HEADER_01X02_SMD_RA" V 3050 6550 50  0000 C CNN
-F 2 "stepper_controller:Header_2_Pin_SMD_RA" H 2850 6600 50  0001 C CNN
+F 2 "stepper_controller_mega:Header_2_Pin_SMD_RA" H 2850 6600 50  0001 C CNN
 F 3 "" H 2950 6700 50  0000 C CNN
 F 4 "digikey" H 3050 6800 60  0001 C CNN "Vendor"
@@
 F 0 "SW1" H 1500 7450 40  0000 L CNN
 F 1 "SPST_SLIDE_AS" H 1350 7625 40  0000 L CNN
-F 2 "stepper_controller:SPST_SLIDE_AS" H 1475 7325 60  0001 C CNN
+F 2 "stepper_controller_mega:SPST_SLIDE_AS" H 1475 7325 60  0001 C CNN
 F 3 "" H 1575 7475 60  0000 C CNN
 F 4 "digikey" H 1675 7725 60  0001 C CNN "Vendor"
@@
 F 0 "C1" H 2850 7600 40  0000 L CNN
 F 1 "10uF" H 2856 7415 40  0000 L CNN
-F 2 "stepper_controller:SM1210" H 2888 7350 30  0001 C CNN
+F 2 "stepper_controller_mega:SM1210" H 2888 7350 30  0001 C CNN
 F 3 "" H 2850 7500 60  0000 C CNN
 F 4 "digikey" H 2950 7700 60  0001 C CNN "Vendor"
@@
 F 0 "IM1" H 7700 3100 60  0000 C CNN
 F 1 "IM483H" H 7350 3100 60  0000 C CNN
-F 2 "stepper_controller:IM483H_IM805H_PR-22" H 7350 3400 60  0001 C CNN
+F 2 "stepper_controller_mega:IM483H_IM805H_PR-22" H 7350 3400 60  0001 C CNN
 F 3 "" H 7650 3100 60  0000 C CNN
 F 4 "schneider" H 7350 3500 60  0001 C CNN "Vendor"
@@
 F 0 "R1" V 5800 2050 40  0000 C CNN
 F 1 "1.69k" V 5700 2050 40  0000 C CNN
-F 2 "stepper_controller:SM1210" V 5630 2050 30  0001 C CNN
+F 2 "stepper_controller_mega:SM1210" V 5630 2050 30  0001 C CNN
 F 3 "" V 5780 2050 30  0000 C CNN
 F 4 "digikey" V 5880 2150 60  0001 C CNN "Vendor"
@@
 F 0 "R2" V 6050 2050 40  0000 C CNN
 F 1 "316" V 5950 2050 40  0000 C CNN
-F 2 "stepper_controller:SM1210" V 5880 2050 30  0001 C CNN
+F 2 "stepper_controller_mega:SM1210" V 5880 2050 30  0001 C CNN
 F 3 "" V 6030 2050 30  0000 C CNN
 F 4 "digikey" V 6130 2150 60  0001 C CNN "Vendor"
